File: Electronics/chicken-shield.brd (EAGLE design)
At the start: 68.6 x 53.3 mm, 11 parts, among them IC1 BD6230F, SW1 SPST_TACT-EVQQ2, SW2 SPST_TACT-EVQQ2

Commit message: Bringing up to date
Parts:
- added BATTERY, PVCELL: (no value), pinhead:1X02
- added OK1: TLP185, opto:MINI-FLAT-4
- added R1: 1K, rcl:M0805
- added R2: 10K, rcl:M0805
- moved SW1 71.3 mm to (58.4, 20.3), turned to 180 degrees
- moved SW2 63.4 mm to (38.7, 20.3), turned to 180 degrees
- moved CORD-SWITCH 44.1 mm to (7.62, 15.2), turned to 270 degrees
- moved MOTOR 37.7 mm to (7.62, 24.8), turned to 270 degrees
- moved R3 35.6 mm to (32.4, 32.4), turned to 180 degrees
- moved IC1 32.9 mm to (20.3, 24.1)
Connections:
- removed net DIG5: PWML.6, SW2.B, SW2.B'
- removed net DIG6: PWML.7, SW1.B, SW1.B'
- removed net DIG7: PWML.8
- new net N$1: OK1.2, PVCELL.1
- new net N$2: OK1.1, R1.2
- new net N$6: PVCELL.2, R1.1
- new net N$7: OK1.4, PWML.6, R2.1
- new net N$8: PWML.8, SW1.B, SW1.B'
- new net N$9: PWML.7, SW2.B, SW2.B'
- net +12V: now also BATTERY.2
- net +5V: now also R2.2
- net DIG2: now also PWML.5; no longer PWML.3
- net DIG4: now also PWML.3; no longer PWML.5
- net GND: now also BATTERY.1, OK1.3, POWER.6, SW1.A
Routing:
- net N$7: track 0.00 -> 53.7 mm
- net N$8: track 0.00 -> 42.0 mm
- net A5: track 37.2 -> 0.00 mm
- net N$4: track 3.17 -> 35.5 mm
- net GND: track 103.0 -> 74.4 mm, vias 6 -> 2
- net N$9: track 0.00 -> 27.4 mm
- net +12V: track 15.1 -> 34.9 mm
- net DIG3: track 0.00 -> 19.7 mm
- net N$5: track 0.00 -> 15.2 mm
- net DIG2: track 42.5 -> 27.4 mm
- net N$3: track 0.00 -> 14.6 mm
- net DIG4: track 0.00 -> 11.9 mm
- net +5V: track 0.00 -> 10.5 mm
- net N$1: track 0.00 -> 8.82 mm
- net N$6: track 0.00 -> 4.66 mm
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Other:
- board size 68.6 x 53.3 mm -> 73 x 53.3 mm
