File: Electronics/chicken-shield.sch (EAGLE design)
At the start: 11 parts, among them IC1 BD6230F, SW1 SPST_TACT-EVQQ2, SW2 SPST_TACT-EVQQ2

Commit message: Bringing up to date
Parts:
- added BATTERY, PVCELL: (no value), pinhead:PINHD-1X2
- added OK1: TLP185, opto:TLP283
- added R1: 1K, rcl:R-EU_M0805
- added R2: 10K, rcl:R-EU_M0805
Connections:
- removed net DIG5: PWML.6, SW2.S, SW2.S1
- removed net DIG6: PWML.7, SW1.S, SW1.S1
- removed net DIG7: PWML.8
- new net N$1: OK1.C, PVCELL.1
- new net N$2: OK1.A, R1.2
- new net N$6: PVCELL.2, R1.1
- new net N$7: OK1.COL, PWML.6, R2.1
- new net N$8: PWML.8, SW1.S, SW1.S1
- new net N$9: PWML.7, SW2.S, SW2.S1
- net +12V: now also BATTERY.2
- net +5V: now also R2.2
- net DIG2: now also PWML.5; no longer PWML.3
- net DIG4: now also PWML.3; no longer PWML.5
- net GND: now also BATTERY.1, OK1.EMIT, POWER.6, SW1.P
Other:
- note added: "GPL"
- note removed: "Creative Commons Attribution Share-Alike 2.5"
